File: kicad/picovga/picovga.kicad_sch (KiCad schematic)
At the start: 26 parts, among them J0 VGA_FEMALE, J1 Micro_SD_Card, U0 PICO_RP2040, U1 PCA9306DC

Commit message: board off for fabrication
Parts:
- J0: footprint Connector_Dsub:DSUB-15-HD_Female_Horizontal_P2.29x1.98mm_EdgePinOffset3.03mm_Housed_MountingHolesOffset4.94mm -> pico:XM4L1542132
Changed lines of the file:
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@@
   (junction (at 176.53 52.705) (diameter 0.9144) (color 0 0 0 0))
   (junction (at 180.975 55.245) (diameter 0.9144) (color 0 0 0 0))
+  (no_connect (at 201.295 117.475))
+  (no_connect (at 47.625 33.655))
+  (no_connect (at 201.295 104.775))
   (no_connect (at 201.295 99.695))
   (no_connect (at 201.295 145.415))
+  (no_connect (at 201.295 109.855))
+  (no_connect (at 201.295 112.395))
+  (no_connect (at 32.385 48.895))
+  (no_connect (at 201.295 120.015))
   (no_connect (at 201.295 122.555))
-  (no_connect (at 201.295 104.775))
-  (no_connect (at 201.295 109.855))
-  (no_connect (at 32.385 48.895))
-  (no_connect (at 201.295 112.395))
-  (no_connect (at 201.295 120.015))
-  (no_connect (at 201.295 117.475))
-  (no_connect (at 47.625 33.655))
   (wire (pts (xy 21.59 97.155) (xy 21.59 100.965))
     (stroke (width 0) (type solid) (color 0 0 0 0))
@@
     (property "Reference" "J0" (id 0) (at 40.005 20.32 0))
     (property "Value" "VGA_FEMALE" (id 1) (at 40.005 22.86 0))
-    (property "Footprint" "Connector_Dsub:DSUB-15-HD_Female_Horizontal_P2.29x1.98mm_EdgePinOffset3.03mm_Housed_MountingHolesOffset4.94mm" (id 2) (at 15.875 33.655 0)
+    (property "Footprint" "pico:XM4L1542132" (id 2) (at 15.875 33.655 0)
       (effects (font (size 1.27 1.27)) hide)
     )
@@
     )
     (path "/fb9eec4d-7fd3-4010-93cd-fb8ede1a382f"
-      (reference "J0") (unit 1) (value "VGA_FEMALE") (footprint "Connector_Dsub:DSUB-15-HD_Female_Horizontal_P2.29x1.98mm_EdgePinOffset3.03mm_Housed_MountingHolesOffset4.94mm")
+      (reference "J0") (unit 1) (value "VGA_FEMALE") (footprint "pico:XM4L1542132")
     )
     (path "/8168f700-c4f5-464a-b86d-c0dd3a1ff03c"
